Commit message: Mergeing updated master

File: kortex_description/grippers/gen3_lite_2f/urdf/gen3_lite_2f.ros2_control.xacro (robot description, xacro)
@@ -9,5 +9,16 @@
         isaac_joint_commands:=/isaac_joint_commands
         isaac_joint_states:=/isaac_joint_states
-        use_internal_bus_gripper_comm:=false">
+        use_internal_bus_gripper_comm:=true
+        gripper_joint_name:=right_finger_bottom_joint
+        tf_prefix:=''
+        robot_ip:=192.168.1.10
+        username:=admin
+        password:=admin
+        port:=10000
+        port_realtime:=10001
+        session_inactivity_timeout_ms:=60000
+        connection_inactivity_timeout_ms:=2000
+        gripper_max_velocity:=100.0
+        gripper_max_force:=100.0">
         <ros2_control name="GripperHardwareInterface" type="system">
             <hardware>
@@ -26,4 +37,19 @@
                     <param name="state_following_offset">0.0</param>
                 </xacro:if>
+                <xacro:unless value="${sim_isaac or sim_ignition or use_fake_hardware}">
+                    <plugin>kortex_driver/KortexMultiInterfaceHardware</plugin>
+                    <param name="robot_ip">${robot_ip}</param>
+                    <param name="username">${username}</param>
+                    <param name="password">${password}</param>
+                    <param name="port">${port}</param>
+                    <param name="port_realtime">${port_realtime}</param>
+                    <param name="session_inactivity_timeout_ms">${session_inactivity_timeout_ms}</param>
+                    <param name="connection_inactivity_timeout_ms">${connection_inactivity_timeout_ms}</param>
+                    <param name="tf_prefix">"${tf_prefix}"</param>
+                    <param name="use_internal_bus_gripper_comm">${use_internal_bus_gripper_comm}</param>
+                    <param name="gripper_joint_name">${gripper_joint_name}</param>
+                    <param name="gripper_max_velocity">${gripper_max_velocity}</param>
+                    <param name="gripper_max_force">${gripper_max_force}</param>
+                </xacro:unless>
             </hardware>
             <!-- Joint interfaces -->
@@ -32,7 +58,9 @@
                 <command_interface name="position" />
                 <state_interface name="position">
-                    <param name="initial_value">0.85</param>
+                    <param name="initial_value">0.0</param>
                 </state_interface>
-                <state_interface name="velocity"/>
+                <state_interface name="velocity">
+                    <param name="initial_value">0.0</param>
+                </state_interface>
             </joint>
             <!-- When simulating we need to include the rest of the gripper joints -->

File: kortex_description/grippers/gen3_lite_2f/urdf/gen3_lite_2f_macro.xacro (robot description, xacro)
@@ -4,4 +4,5 @@
     parent
     prefix
+    com_port
     use_fake_hardware:=false
     mock_sensor_commands:=false
@@ -11,14 +12,4 @@
     isaac_joint_states:=/isaac_joint_states
     use_internal_bus_gripper_comm:=true">
-    <xacro:include filename="$(find kortex_description)/grippers/gen3_lite_2f/urdf/gen3_lite_2f.ros2_control.xacro" />
-    <xacro:gripper_ros2_control
-      prefix="${prefix}"
-      use_fake_hardware="${use_fake_hardware}"
-      mock_sensor_commands="${mock_sensor_commands}"
-      sim_ignition="${sim_ignition}"
-      sim_isaac="${sim_isaac}"
-      isaac_joint_commands="${isaac_joint_commands}"
-      isaac_joint_states="${isaac_joint_states}"
-      use_internal_bus_gripper_comm="${use_internal_bus_gripper_comm}"/>
     <!-- Tool frame used by the arm -->
     <link name="${prefix}tool_frame"/>
@@ -45,5 +36,5 @@
         <origin xyz="0 0 0" rpy="0 0 0" />
         <geometry>
-          <mesh filename="package://kortex_description/grippers/gen3_lite_2f/meshes/gripper_base_link.STL" />
+          <mesh filename="file://$(find kortex_description)/grippers/gen3_lite_2f/meshes/gripper_base_link.STL" />
         </geometry>
         <material name="">
@@ -54,5 +45,5 @@
         <origin xyz="0 0 0" rpy="0 0 0" />
         <geometry>
-          <mesh filename="package://kortex_description/grippers/gen3_lite_2f/meshes/gripper_base_link.STL" />
+          <mesh filename="file://$(find kortex_description)/grippers/gen3_lite_2f/meshes/gripper_base_link.STL" />
         </geometry>
       </collision>
@@ -70,5 +61,5 @@
       <origin xyz="0 0 0" rpy="0 0 0" />
       <geometry>
-        <mesh filename="package://kortex_description/grippers/gen3_lite_2f/meshes/right_finger_prox_link.STL" />
+        <mesh filename="file://$(find kortex_description)/grippers/gen3_lite_2f/meshes/right_finger_prox_link.STL" />
       </geometry>
       <material name="">
@@ -79,5 +70,5 @@
       <origin xyz="0 0 0" rpy="0 0 0" />
       <geometry>
-        <mesh filename="package://kortex_description/grippers/gen3_lite_2f/meshes/right_finger_prox_link.STL" />
+        <mesh filename="file://$(find kortex_description)/grippers/gen3_lite_2f/meshes/right_finger_prox_link.STL" />
       </geometry>
     </collision>
@@ -92,5 +83,5 @@
       <child link="${prefix}right_finger_prox_link" />
       <axis xyz="0 0 -1" />
-      <limit lower="0.0" upper="0.85" effort="1000" velocity="0.6" />
+      <limit lower="0.0" upper="0.85" effort="50" velocity="0.6" />
     </joint>
     <link name="${prefix}right_finger_dist_link">
@@ -103,5 +94,5 @@
         <origin xyz="0 0 0" rpy="0 0 0" />
         <geometry>
-          <mesh filename="package://kortex_description/grippers/gen3_lite_2f/meshes/right_finger_dist_link.STL" />
+          <mesh filename="file://$(find kortex_description)/grippers/gen3_lite_2f/meshes/right_finger_dist_link.STL" />
         </geometry>
         <material name="">
@@ -112,5 +103,5 @@
         <origin xyz="0 0 0" rpy="0 0 0" />
         <geometry>
-          <mesh filename="package://kortex_description/grippers/gen3_lite_2f/meshes/right_finger_dist_link.STL" />
+          <mesh filename="file://$(find kortex_description)/grippers/gen3_lite_2f/meshes/right_finger_dist_link.STL" />
         </geometry>
       </collision>
@@ -136,5 +127,5 @@
         <origin xyz="0 0 0" rpy="0 0 0" />
         <geometry>
-          <mesh filename="package://kortex_description/grippers/gen3_lite_2f/meshes/left_finger_prox_link.STL" />
+          <mesh filename="file://$(find kortex_description)/grippers/gen3_lite_2f/meshes/left_finger_prox_link.STL" />
         </geometry>
         <material name="">
@@ -145,5 +136,5 @@
         <origin xyz="0 0 0" rpy="0 0 0" />
         <geometry>
-          <mesh filename="package://kortex_description/grippers/gen3_lite_2f/meshes/left_finger_prox_link.STL" />
+          <mesh filename="file://$(find kortex_description)/grippers/gen3_lite_2f/meshes/left_finger_prox_link.STL" />
         </geometry>
       </collision>
@@ -169,5 +160,5 @@
         <origin xyz="0 0 0" rpy="0 0 0" />
         <geometry>
-          <mesh filename="package://kortex_description/grippers/gen3_lite_2f/meshes/left_finger_dist_link.STL" />
+          <mesh filename="file://$(find kortex_description)/grippers/gen3_lite_2f/meshes/left_finger_dist_link.STL" />
         </geometry>
         <material name="">
@@ -178,5 +169,5 @@
         <origin xyz="0 0 0" rpy="0 0 0" />
         <geometry>
-          <mesh filename="package://kortex_description/grippers/gen3_lite_2f/meshes/left_finger_dist_link.STL" />
+          <mesh filename="file://$(find kortex_description)/grippers/gen3_lite_2f/meshes/left_finger_dist_link.STL" />
         </geometry>
       </collision>

File: kortex_description/grippers/robotiq_2f_140/urdf/robotiq_2f_140_macro.xacro (robot description, xacro)
@@ -5,6 +5,11 @@
     prefix
     use_fake_hardware:=false
+<<<<<<< HEAD
     mock_sensor_commands:=false
     sim_ignition:=false
+=======
+    fake_sensor_commands:=false
+    sim_gazebo:=false
+>>>>>>> 7ad1cc1 (Mergeing updated master)
     sim_isaac:=false
     isaac_joint_commands:=/isaac_joint_commands
@@ -25,6 +30,11 @@
         com_port="${com_port}"
         use_fake_hardware="${use_fake_hardware}"
+<<<<<<< HEAD
         mock_sensor_commands="${mock_sensor_commands}"
         sim_ignition="${sim_ignition}"
+=======
+        mock_sensor_commands="${fake_sensor_commands}"
+        sim_gazebo="${sim_gazebo}"
+>>>>>>> 7ad1cc1 (Mergeing updated master)
         sim_isaac="${sim_isaac}"
         isaac_joint_commands="${isaac_joint_commands}"
